File: containment/containment-simple.sch (KiCad schematic (older format))
At the start: 36 parts, among them J1 Conn_02x05_Odd_Even, J3 Conn_01x02, J4 Conn_01x02, J5 Conn_01x02, J6 Conn_01x02, Q1 BSS84, Q2 BSS84, Q3 BSS84, Q4 BSS84, U1 TMP411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

Commit message: add spixes
Parts:
- added JEXP1, JFLUID1, JPUMP1, JPUMP2: Conn_01x02, Connector_PinHeader_2.54mm:PinHeader_1x02_P2.54mm_Horizontal, symbol Connector_Generic:Conn_01x02
- added U3, U4: SFH617A-1, Package_DIP:DIP-4_W7.62mm, symbol Isolator:SFH617A-1
- JSOL1: renamed from J3; footprint Connector_PinHeader_2.54mm:PinHeader_1x02_P2.54mm_Vertical -> Connector_PinHeader_2.54mm:PinHeader_1x02_P2.54mm_Horizontal
- JSOL2: renamed from J4; footprint Connector_PinHeader_2.54mm:PinHeader_1x02_P2.54mm_Vertical -> Connector_PinHeader_2.54mm:PinHeader_1x02_P2.54mm_Horizontal
- JSOL3: renamed from J5; footprint Connector_PinHeader_2.54mm:PinHeader_1x02_P2.54mm_Vertical -> Connector_PinHeader_2.54mm:PinHeader_1x02_P2.54mm_Horizontal
- JSOL4: renamed from J6; footprint Connector_PinHeader_2.54mm:PinHeader_1x02_P2.54mm_Vertical -> Connector_PinHeader_2.54mm:PinHeader_1x02_P2.54mm_Horizontal
- JTEMP1: footprint Connector_PinHeader_2.54mm:PinHeader_1x02_P2.54mm_Vertical -> Connector_PinHeader_2.54mm:PinHeader_1x02_P2.54mm_Horizontal
Connections:
- net labels added: HV+, HV-, experiment+, experiment-
- wire segments 71 -> 77
- no-connect marks 5 -> 1
Other:
- moved on the sheet: J1

Commit message: spikey 2
Parts:
- removed JFLUID1: Conn_01x02, Connector_PinHeader_2.54mm:PinHeader_1x02_P2.54mm_Horizontal, symbol Connector_Generic:Conn_01x02
- added JFLUID1, JFLUID2: Conn_01x03, symbol Connector_Generic:Conn_01x03
Connections:
- wire segments 77 -> 81
Changed lines of the file:
@@
 Wire Wire Line
 	4500 3500 4650 3500
-Text Label 8100 3400 2    50   ~ 0
+Text Label 8550 2600 2    50   ~ 0
 p0
 Text Label 1200 1900 2    50   ~ 0
@@
 Wire Wire Line
 	4500 4350 4650 4350
-Text Label 8100 3300 2    50   ~ 0
+Text Label 8550 3250 2    50   ~ 0
 p1
 $Comp
@@
 Text Label 5250 4350 0    50   ~ 0
 HV-
-$Comp
-L Connector_Generic:Conn_01x02 JFLUID1
-U 1 1 5FE34B2D
-P 8300 3300
-F 0 "JFLUID1" H 8380 3292 50  0000 L CNN
-F 1 "Conn_01x02" H 8380 3201 50  0000 L CNN
-F 2 "Connector_PinHeader_2.54mm:PinHeader_1x02_P2.54mm_Horizontal" H 8300 3300 50  0001 C CNN
-F 3 "~" H 8300 3300 50  0001 C CNN
-	1    8300 3300
-	1    0    0    -1
-$EndComp
 Text Label 4650 3300 2    50   ~ 0
 p2
@@
 Text Label 8100 3950 2    50   ~ 0
 experiment-
+$Comp
+L Connector_Generic:Conn_01x03 JFLUID2
+U 1 1 5FECF68D
+P 8750 3350
+F 0 "JFLUID2" H 8830 3392 50  0000 L CNN
+F 1 "Conn_01x03" H 8830 3301 50  0000 L CNN
+F 2 "" H 8750 3350 50  0001 C CNN
+F 3 "~" H 8750 3350 50  0001 C CNN
+	1    8750 3350
+	1    0    0    -1
+$EndComp
+$Comp
+L Connector_Generic:Conn_01x03 JFLUID1
+U 1 1 5FED0BBF
+P 8750 2700
+F 0 "JFLUID1" H 8830 2742 50  0000 L CNN
+F 1 "Conn_01x03" H 8830 2651 50  0000 L CNN
+F 2 "" H 8750 2700 50  0001 C CNN
+F 3 "~" H 8750 2700 50  0001 C CNN
+	1    8750 2700
+	1    0    0    -1
+$EndComp
+$Comp
+L power:+5V #PWR?
+U 1 1 5FED5DAE
+P 8250 2650
+F 0 "#PWR?" H 8250 2500 50  0001 C CNN
+F 1 "+5V" H 8265 2823 50  0000 C CNN
+F 2 "" H 8250 2650 50  0001 C CNN
+F 3 "" H 8250 2650 50  0001 C CNN
+	1    8250 2650
+	1    0    0    -1
+$EndComp
+$Comp
+L power:+5V #PWR?
+U 1 1 5FED5FD2
+P 8200 3250
+F 0 "#PWR?" H 8200 3100 50  0001 C CNN
+F 1 "+5V" H 8215 3423 50  0000 C CNN
+F 2 "" H 8200 3250 50  0001 C CNN
+F 3 "" H 8200 3250 50  0001 C CNN
+	1    8200 3250
+	1    0    0    -1
+$EndComp
+Wire Wire Line
+	8200 3250 8200 3350
+Wire Wire Line
+	8200 3350 8550 3350
+Wire Wire Line
+	8250 2650 8250 2700
+Wire Wire Line
+	8250 2700 8550 2700
+$Comp
+L power:GND #PWR?
+U 1 1 5FEDAF9D
+P 8550 2800
+F 0 "#PWR?" H 8550 2550 50  0001 C CNN
+F 1 "GND" H 8555 2627 50  0000 C CNN
+F 2 "" H 8550 2800 50  0001 C CNN
+F 3 "" H 8550 2800 50  0001 C CNN
+	1    8550 2800
+	1    0    0    -1
+$EndComp
+$Comp
+L power:GND #PWR?
+U 1 1 5FEDBEE4
+P 8550 3450
+F 0 "#PWR?" H 8550 3200 50  0001 C CNN
+F 1 "GND" H 8555 3277 50  0000 C CNN
+F 2 "" H 8550 3450 50  0001 C CNN
+F 3 "" H 8550 3450 50  0001 C CNN
+	1    8550 3450
+	1    0    0    -1
+$EndComp
 $EndSCHEMATC

Commit message: use the correct optocoupler
Parts:
- removed U3, U4: SFH617A-1, Package_DIP:DIP-4_W7.62mm, symbol Isolator:SFH617A-1
- added R10, R11: 470, Resistor_SMD:R_0603_1608Metric, symbol Device:R
- added U3, U4: TLP175A, Package_SO:MFSOP6-4_4.4x3.6mm_P1.27mm, symbol Relay_SolidState:TLP175A
- JFLUID1, JFLUID2: footprint (none) -> Connector_PinHeader_2.54mm:PinHeader_1x03_P2.54mm_Horizontal
Connections:
- wire segments 81 -> 85
Other:
- note added: "Actually TLP172GM"
Changed lines of the file:
@@
-$EndComp
-$Comp
-L Isolator:SFH617A-1 U3
-U 1 1 5FE18190
-P 4950 3400
-F 0 "U3" H 4950 3725 50  0000 C CNN
-F 1 "SFH617A-1" H 4950 3634 50  0000 C CNN
-F 2 "Package_DIP:DIP-4_W7.62mm" H 4750 3200 50  0001 L CIN
-F 3 "http://www.vishay.com/docs/83740/sfh617a.pdf" H 4950 3400 50  0001 L CNN
-	1    4950 3400
-	1    0    0    -1
 $EndComp
 $Comp
@@
 HV-
 $Comp
-L Isolator:SFH617A-1 U4
-U 1 1 5FE2F03C
-P 4950 4250
-F 0 "U4" H 4950 4575 50  0000 C CNN
-F 1 "SFH617A-1" H 4950 4484 50  0000 C CNN
-F 2 "Package_DIP:DIP-4_W7.62mm" H 4750 4050 50  0001 L CIN
-F 3 "http://www.vishay.com/docs/83740/sfh617a.pdf" H 4950 4250 50  0001 L CNN
-	1    4950 4250
-	1    0    0    -1
-$EndComp
-$Comp
 L power:GND #PWR0128
 U 1 1 5FE2F042
@@
 Text Label 5250 4350 0    50   ~ 0
 HV-
-Text Label 4650 3300 2    50   ~ 0
+Text Label 4100 3300 2    50   ~ 0
 p2
-Text Label 4650 4150 2    50   ~ 0
+Text Label 4050 4150 2    50   ~ 0
 p3
 $Comp
@@
 F 0 "JFLUID2" H 8830 3392 50  0000 L CNN
 F 1 "Conn_01x03" H 8830 3301 50  0000 L CNN
-F 2 "" H 8750 3350 50  0001 C CNN
+F 2 "Connector_PinHeader_2.54mm:PinHeader_1x03_P2.54mm_Horizontal" H 8750 3350 50  0001 C CNN
 F 3 "~" H 8750 3350 50  0001 C CNN
 	1    8750 3350
@@
 F 0 "JFLUID1" H 8830 2742 50  0000 L CNN
 F 1 "Conn_01x03" H 8830 2651 50  0000 L CNN
-F 2 "" H 8750 2700 50  0001 C CNN
+F 2 "Connector_PinHeader_2.54mm:PinHeader_1x03_P2.54mm_Horizontal" H 8750 2700 50  0001 C CNN
 F 3 "~" H 8750 2700 50  0001 C CNN
 	1    8750 2700
@@
 $EndComp
 $Comp
-L power:+5V #PWR?
+L power:+5V #PWR0129
 U 1 1 5FED5DAE
 P 8250 2650
-F 0 "#PWR?" H 8250 2500 50  0001 C CNN
+F 0 "#PWR0129" H 8250 2500 50  0001 C CNN
 F 1 "+5V" H 8265 2823 50  0000 C CNN
 F 2 "" H 8250 2650 50  0001 C CNN
@@
 $EndComp
 $Comp
-L power:+5V #PWR?
+L power:+5V #PWR0130
 U 1 1 5FED5FD2
 P 8200 3250
-F 0 "#PWR?" H 8200 3100 50  0001 C CNN
+F 0 "#PWR0130" H 8200 3100 50  0001 C CNN
 F 1 "+5V" H 8215 3423 50  0000 C CNN
 F 2 "" H 8200 3250 50  0001 C CNN
@@
 	8250 2700 8550 2700
 $Comp
-L power:GND #PWR?
+L power:GND #PWR0131
 U 1 1 5FEDAF9D
 P 8550 2800
-F 0 "#PWR?" H 8550 2550 50  0001 C CNN
+F 0 "#PWR0131" H 8550 2550 50  0001 C CNN
 F 1 "GND" H 8555 2627 50  0000 C CNN
 F 2 "" H 8550 2800 50  0001 C CNN
@@
 $EndComp
 $Comp
-L power:GND #PWR?
+L power:GND #PWR0132
 U 1 1 5FEDBEE4
 P 8550 3450
-F 0 "#PWR?" H 8550 3200 50  0001 C CNN
+F 0 "#PWR0132" H 8550 3200 50  0001 C CNN
 F 1 "GND" H 8555 3277 50  0000 C CNN
 F 2 "" H 8550 3450 50  0001 C CNN
@@
 	1    0    0    -1
 $EndComp
+$Comp
+L Device:R R10
+U 1 1 5FF82983
+P 4400 3300
+F 0 "R10" V 4193 3300 50  0000 C CNN
+F 1 "470" V 4284 3300 50  0000 C CNN
+F 2 "Resistor_SMD:R_0603_1608Metric" V 4330 3300 50  0001 C CNN
+F 3 "~" H 4400 3300 50  0001 C CNN
+F 4 "C491208" H 4400 3300 50  0001 C CNN "LCSC"
+	1    4400 3300
+	0    1    1    0
+$EndComp
+$Comp
+L Device:R R11
+U 1 1 5FF82CDB
+P 4350 4150
+F 0 "R11" V 4143 4150 50  0000 C CNN
+F 1 "470" V 4234 4150 50  0000 C CNN
+F 2 "Resistor_SMD:R_0603_1608Metric" V 4280 4150 50  0001 C CNN
+F 3 "~" H 4350 4150 50  0001 C CNN
+F 4 "C491208" H 4350 4150 50  0001 C CNN "LCSC"
+	1    4350 4150
+	0    1    1    0
+$EndComp
+Wire Wire Line
+	4200 4150 4050 4150
+Wire Wire Line
+	4500 4150 4650 4150
+Wire Wire Line
+	4550 3300 4650 3300
+Wire Wire Line
+	4250 3300 4100 3300
+Text Notes 4650 2950 0    50   ~ 0
+Actually TLP172GM
+$Comp
+L Relay_SolidState:TLP175A U3
+U 1 1 5FFC94E5
+P 4950 3400
+F 0 "U3" H 4950 3725 50  0000 C CNN
+F 1 "TLP175A" H 4950 3634 50  0000 C CNN
+F 2 "Package_SO:MFSOP6-4_4.4x3.6mm_P1.27mm" H 4950 3100 50  0001 C CIN
+F 3 "https://toshiba.semicon-storage.com/info/docget.jsp?did=13665&prodName=TLP175A" H 4950 3400 50  0001 L CNN
+F 4 "C261926" H 4950 3400 50  0001 C CNN "LCSC"
+	1    4950 3400
+	1    0    0    -1
+$EndComp
+$Comp
+L Relay_SolidState:TLP175A U4
+U 1 1 5FFD1C88
+P 4950 4250
+F 0 "U4" H 4950 4575 50  0000 C CNN
+F 1 "TLP175A" H 4950 4484 50  0000 C CNN
+F 2 "Package_SO:MFSOP6-4_4.4x3.6mm_P1.27mm" H 4950 3950 50  0001 C CIN
+F 3 "https://toshiba.semicon-storage.com/info/docget.jsp?did=13665&prodName=TLP175A" H 4950 4250 50  0001 L CNN
+F 4 "C261926" H 4950 4250 50  0001 C CNN "LCSC"
+	1    4950 4250
+	1    0    0    -1
+$EndComp
