File: containment/containment-simple.sch (KiCad schematic (older format))
At the start: 45 parts, among them J1 Conn_02x05_Odd_Even, Q1 BSS84, Q2 BSS84, Q3 BSS84, Q4 BSS84, U1 TMP411, U2 PCA9557, U3 TLP175A, U4 TLP175A

Commit message: inner containment baord lookin pretty good
Parts:
- removed D2: D, Diode_SMD:D_SOD-123, symbol Device:D
- removed D3: LED, LED_SMD:LED_1206_3216Metric, symbol Device:LED
- removed JFLUID1, JFLUID2: Conn_01x03, Connector_PinHeader_2.54mm:PinHeader_1x03_P2.54mm_Horizontal, symbol Connector_Generic:Conn_01x03
- removed JSOL1: Conn_01x02, Connector_PinHeader_2.54mm:PinHeader_1x02_P2.54mm_Horizontal, symbol Connector_Generic:Conn_01x02
- removed R2: 1k, Resistor_SMD:R_0603_1608Metric, symbol Device:R
- removed R6: 10k, Resistor_SMD:R_0603_1608Metric, symbol Device:R
- C1: LCSC C77055 -> C14663
- C3: LCSC C14860 -> C13585
- D1, D5, D7, D9: footprint LED_SMD:LED_1206_3216Metric -> LED_SMD:LED_0603_1608Metric; LCSC C264549 -> C2286
- D4, D6, D8: footprint Diode_SMD:D_SOD-123 -> Diode_SMD:D_SOD-323F; LCSC C222352 -> C2128
- JEXP1, JPUMP1, JPUMP2, JSOL2, JSOL3, JSOL4, JTEMP1: footprint Connector_PinHeader_2.54mm:PinHeader_1x02_P2.54mm_Horizontal -> Connector_JST:JST_PH_S2B-PH-K_1x02_P2.00mm_Horizontal
- R1, R3, R4, R5: LCSC C50069 -> C21190
- R10, R11: LCSC C491208 -> C23179
- R7, R8, R9: LCSC C491175 -> C25804
Connections:
- net labels added: experiment
- net labels removed: experiment+, experiment-
- wire segments 85 -> 71
- no-connect marks 1 -> 0
Other:
- moved on the sheet: C1, C3, JEXP1, JPUMP1, JPUMP2, JTEMP1, R10, R11, U1

Commit message: ordered it supposedly
Parts:
- Q1, Q2, Q3, Q4: LCSC C508197 -> C10487
- renumbered JSOL2 to JSOL1, JSOL3 to JSOL2, JSOL4 to JSOL3
Other:
- note added: "Don't need a pullup on p4 --\ninitial state doesn't matter as\nlong as pump driver is off"
Changed lines of the file:
@@
 $EndComp
 Connection ~ 2200 1700
-$Comp
-L power:+5V #PWR0116
-U 1 1 5F266259
-P 7000 900
-F 0 "#PWR0116" H 7000 750 50  0001 C CNN
-F 1 "+5V" H 7015 1073 50  0000 C CNN
-F 2 "" H 7000 900 50  0001 C CNN
-F 3 "" H 7000 900 50  0001 C CNN
-	1    7000 900
-	1    0    0    -1
-$EndComp
 Wire Wire Line
 	7000 900  7000 1000
@@
 F 2 "Package_TO_SOT_SMD:SOT-23" H 4250 5775 50  0001 L CIN
 F 3 "http://assets.nexperia.com/documents/data-sheet/BSS84.pdf" H 4050 5850 50  0001 L CNN
-F 4 "C508197" H 4050 5850 50  0001 C CNN "LCSC"
+F 4 "C10487" H 4050 5850 50  0001 C CNN "LCSC"
 	1    4050 5850
-	1    0    0    -1
+	1    0    0    1
 $EndComp
 $Comp
@@
 F 2 "Package_TO_SOT_SMD:SOT-23" H 10150 1125 50  0001 L CIN
 F 3 "http://assets.nexperia.com/documents/data-sheet/BSS84.pdf" H 9950 1200 50  0001 L CNN
-F 4 "C508197" H 9950 1200 50  0001 C CNN "LCSC"
+F 4 "C10487" H 9950 1200 50  0001 C CNN "LCSC"
 	1    9950 1200
 	1    0    0    1
@@
 F 2 "Package_TO_SOT_SMD:SOT-23" H 7450 1125 50  0001 L CIN
 F 3 "http://assets.nexperia.com/documents/data-sheet/BSS84.pdf" H 7250 1200 50  0001 L CNN
-F 4 "C508197" H 7250 1200 50  0001 C CNN "LCSC"
+F 4 "C10487" H 7250 1200 50  0001 C CNN "LCSC"
 	1    7250 1200
 	1    0    0    1
@@
 $EndComp
 $Comp
-L Connector_Generic:Conn_01x02 JSOL3
+L Connector_Generic:Conn_01x02 JSOL2
 U 1 1 5F2698C2
 P 8200 1600
-F 0 "JSOL3" H 8118 1817 50  0000 C CNN
+F 0 "JSOL2" H 8118 1817 50  0000 C CNN
 F 1 "Conn_01x02" H 8118 1726 50  0000 C CNN
 F 2 "Connector_JST:JST_PH_S2B-PH-K_1x02_P2.00mm_Horizontal" H 8200 1600 50  0001 C CNN
@@
 F 2 "Package_TO_SOT_SMD:SOT-23" H 8800 1125 50  0001 L CIN
 F 3 "http://assets.nexperia.com/documents/data-sheet/BSS84.pdf" H 8600 1200 50  0001 L CNN
-F 4 "C508197" H 8600 1200 50  0001 C CNN "LCSC"
+F 4 "C10487" H 8600 1200 50  0001 C CNN "LCSC"
 	1    8600 1200
 	1    0    0    1
@@
 $EndComp
 $Comp
-L Connector_Generic:Conn_01x02 JSOL2
+L Connector_Generic:Conn_01x02 JSOL1
 U 1 1 5F266275
 P 6850 1600
-F 0 "JSOL2" H 6768 1817 50  0000 C CNN
+F 0 "JSOL1" H 6768 1817 50  0000 C CNN
 F 1 "Conn_01x02" H 6768 1726 50  0000 C CNN
 F 2 "Connector_JST:JST_PH_S2B-PH-K_1x02_P2.00mm_Horizontal" H 6850 1600 50  0001 C CNN
@@
 $EndComp
 $Comp
-L Connector_Generic:Conn_01x02 JSOL4
+L Connector_Generic:Conn_01x02 JSOL3
 U 1 1 5F26C725
 P 9550 1600
-F 0 "JSOL4" H 9468 1817 50  0000 C CNN
+F 0 "JSOL3" H 9468 1817 50  0000 C CNN
 F 1 "Conn_01x02" H 9468 1726 50  0000 C CNN
 F 2 "Connector_JST:JST_PH_S2B-PH-K_1x02_P2.00mm_Horizontal" H 9550 1600 50  0001 C CNN
@@
 	1    0    0    -1
 $EndComp
+Text Notes 4200 850  0    50   ~ 0
+Don't need a pullup on p4 --\ninitial state doesn't matter as\nlong as pump driver is off
+$Comp
+L power:+12V #PWR?
+U 1 1 606B96E5
+P 7000 900
+F 0 "#PWR?" H 7000 750 50  0001 C CNN
+F 1 "+12V" H 7015 1073 50  0000 C CNN
+F 2 "" H 7000 900 50  0001 C CNN
+F 3 "" H 7000 900 50  0001 C CNN
+	1    7000 900
+	1    0    0    -1
+$EndComp

Commit message: containment schematic updated to include experiment & correct voltage on valve mosfets
Parts:
- removed JEXP1: Conn_01x02, Connector_JST:JST_PH_S2B-PH-K_1x02_P2.00mm_Horizontal, symbol Connector_Generic:Conn_01x02
- added Q7, Q8, Q9: BC846, Package_TO_SOT_SMD:SOT-23, symbol Transistor_BJT:BC846
- added R21, R22, R23: 10k, Resistor_SMD:R_0603_1608Metric, symbol Device:R
- JPUMP1, JPUMP2, JSOL1, JSOL2, JSOL3, JTEMP1: footprint Connector_JST:JST_PH_S2B-PH-K_1x02_P2.00mm_Horizontal -> Connector_JST:JST_PH_B2B-PH-K_1x02_P2.00mm_Vertical
- R7, R8, R9: LCSC C25804 -> (none)
Connections:
- net labels added: p0_fluid_1_hi, p1_fluid_1_lo, p2_fluid_2_hi_expctl, p3_fluid_2_lo_expctl, p4_pump_select, p5_sol1, p6_sol1, p6_sol2, p7_sol3
- net labels removed: p0, p1, p2, p3, p4, p5, p6, p7
- wire segments 71 -> 73
Other:
- moved on the sheet: D4, D5, D6, D7, D8, D9, JSOL1, JSOL2, JSOL3, Q2, Q3, Q4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
