File: containment/fluid-sensors.sch (KiCad schematic (older format))
At the start: 24 parts

Commit message: inner containment baord lookin pretty good
Parts:
- removed R? (x3): R, symbol Device:R
- removed U? (x2): LM339, symbol Analog_DAC:DAC081C081CIMK
- removed U? (x3): LM339, symbol Amplifier_Operational:LM358
- added C2, C4, C5: .1uF, Capacitor_SMD:C_0603_1608Metric, symbol Device:C
- added U5: LM358, Package_SO:SOIC-8_3.9x4.9mm_P1.27mm, symbol Amplifier_Operational:LM358
- added U7, U8: MCP4725xxx-xCH, Package_TO_SOT_SMD:SOT-23-6, symbol Analog_DAC:MCP4725xxx-xCH
- J2, J3: renamed from J?; value Conn_01x04 -> Conn_01x03; footprint (none) -> Connector_JST:JST_PH_S3B-PH-K_1x03_P2.00mm_Horizontal; symbol Connector_Generic:Conn_01x04 -> Connector_Generic:Conn_01x03
- Q5, Q6: renamed from Q?; LCSC (none) -> C31776
- R12, R14, R15, R16, R20: renamed from R?; value R -> 10k; footprint (none) -> Resistor_SMD:R_0603_1608Metric; LCSC (none) -> C25804
- R13, R18: renamed from R?; value R -> 50; footprint (none) -> Resistor_SMD:R_0603_1608Metric; LCSC (none) -> C22809
- U6: renamed from U?; footprint (none) -> Package_SO:TSSOP-14_4.4x5mm_P0.65mm; LCSC (none) -> C42184
Connections:
- net labels added: 1_3rds, 2_3rds
- wire segments 52 -> 57
- no-connect marks 2 -> 0
Other:
- note added: "358 max output: 3.3V"
- note added: "Pin-compatible with some others (eg, DAC5571)\nbut double check! esp. gnd and vcc"

Commit message: can i get a go dawgs
Parts:
- added C?: .1uF, symbol Device:C
- added R? (x2): 10k, symbol Device:R
- added R? (x2): R, symbol Device:R
- renumbered J2 to JFLUID1, J3 to JFLUID2
Connections:
- wire segments 57 -> 67
Other:
- moved on the sheet: R16
Changed lines of the file:
@@
 L Device:R R16
 U 1 1 603018B3
-P 5450 3150
-F 0 "R16" H 5520 3196 50  0000 L CNN
-F 1 "10k" H 5520 3105 50  0000 L CNN
-F 2 "Resistor_SMD:R_0603_1608Metric" V 5380 3150 50  0001 C CNN
-F 3 "~" H 5450 3150 50  0001 C CNN
-F 4 "C25804" H 5450 3150 50  0001 C CNN "LCSC"
-	1    5450 3150
+P 5450 3200
+F 0 "R16" H 5520 3246 50  0000 L CNN
+F 1 "10k" H 5520 3155 50  0000 L CNN
+F 2 "Resistor_SMD:R_0603_1608Metric" V 5380 3200 50  0001 C CNN
+F 3 "~" H 5450 3200 50  0001 C CNN
+F 4 "C25804" H 5450 3200 50  0001 C CNN "LCSC"
+	1    5450 3200
 	1    0    0    -1
 $EndComp
@@
 	5450 2750 5450 2800
 Wire Wire Line
-	5450 3300 5450 3450
+	5450 3350 5450 3450
 $Comp
 L power:GND #PWR0139
@@
 	1    0    0    -1
 $EndComp
-Text HLabel 6500 2350 2    50   Input ~ 0
+Text HLabel 6850 2350 2    50   Input ~ 0
 sensor_1_hi
-Text HLabel 6500 2900 2    50   Input ~ 0
+Text HLabel 6850 2900 2    50   Input ~ 0
 sensor_1_lo
 $Comp
-L Connector_Generic:Conn_01x03 J3
+L Connector_Generic:Conn_01x03 JFLUID2
 U 1 1 60315D85
 P 5350 4350
-F 0 "J3" H 5430 4342 50  0000 L CNN
+F 0 "JFLUID2" H 5430 4342 50  0000 L CNN
 F 1 "Conn_01x03" H 5430 4251 50  0000 L CNN
 F 2 "Connector_JST:JST_PH_S3B-PH-K_1x03_P2.00mm_Horizontal" H 5350 4350 50  0001 C CNN
@@
 	1    0    0    -1
 $EndComp
-Text HLabel 6800 5400 2    50   Input ~ 0
+Text HLabel 7150 5400 2    50   Input ~ 0
 sensor_2_hi
-Text HLabel 6800 5950 2    50   Input ~ 0
+Text HLabel 7150 5950 2    50   Input ~ 0
 sensor_2_lo
 $Comp
@@
 Wire Wire Line
 	5900 2800 5450 2800
-Connection ~ 5450 2800
-Wire Wire Line
-	5450 2800 5450 3000
 Connection ~ 4600 3000
-Wire Wire Line
-	4600 3000 5900 3000
 Wire Wire Line
 	4900 6050 6200 6050
@@
 1_3rds
 $Comp
-L Connector_Generic:Conn_01x03 J2
+L Connector_Generic:Conn_01x03 JFLUID1
 U 1 1 602E59B9
 P 5050 1300
-F 0 "J2" H 5130 1292 50  0000 L CNN
+F 0 "JFLUID1" H 5130 1292 50  0000 L CNN
 F 1 "Conn_01x03" H 5130 1201 50  0000 L CNN
 F 2 "Connector_JST:JST_PH_S3B-PH-K_1x03_P2.00mm_Horizontal" H 5050 1300 50  0001 C CNN
@@
 Wire Wire Line
 	7150 1250 6800 1250
+$Comp
+L Device:C C?
+U 1 1 605BF183
+P 5150 3200
+F 0 "C?" H 5265 3246 50  0000 L CNN
+F 1 ".1uF" H 5265 3155 50  0000 L CNN
+F 2 "" H 5188 3050 50  0001 C CNN
+F 3 "~" H 5150 3200 50  0001 C CNN
+	1    5150 3200
+	1    0    0    -1
+$EndComp
+Wire Wire Line
+	5150 3050 5450 3050
+Wire Wire Line
+	4600 3000 5900 3000
+Wire Wire Line
+	5450 3050 5450 2800
+Connection ~ 5450 3050
+Connection ~ 5450 2800
+Wire Wire Line
+	5150 3350 5450 3350
+Connection ~ 5450 3350
+Wire Wire Line
+	6500 2900 6650 2900
+Wire Wire Line
+	6500 2350 6650 2350
+$Comp
+L Device:R R?
+U 1 1 605CB52E
+P 6650 2200
+F 0 "R?" H 6720 2246 50  0000 L CNN
+F 1 "10k" H 6720 2155 50  0000 L CNN
+F 2 "" V 6580 2200 50  0001 C CNN
+F 3 "~" H 6650 2200 50  0001 C CNN
+	1    6650 2200
+	1    0    0    -1
+$EndComp
+Connection ~ 6650 2350
+Wire Wire Line
+	6650 2350 6850 2350
+$Comp
+L Device:R R?
+U 1 1 605CB817
+P 6650 2750
+F 0 "R?" H 6720 2796 50  0000 L CNN
+F 1 "10k" H 6720 2705 50  0000 L CNN
+F 2 "" V 6580 2750 50  0001 C CNN
+F 3 "~" H 6650 2750 50  0001 C CNN
+	1    6650 2750
+	1    0    0    -1
+$EndComp
+Connection ~ 6650 2900
+Wire Wire Line
+	6650 2900 6850 2900
+$Comp
+L power:+5V #PWR?
+U 1 1 605CC9CB
+P 6650 2050
+F 0 "#PWR?" H 6650 1900 50  0001 C CNN
+F 1 "+5V" H 6665 2223 50  0000 C CNN
+F 2 "" H 6650 2050 50  0001 C CNN
+F 3 "" H 6650 2050 50  0001 C CNN
+	1    6650 2050
+	1    0    0    -1
+$EndComp
+$Comp
+L power:+5V #PWR?
+U 1 1 605CCCAA
+P 6650 2600
+F 0 "#PWR?" H 6650 2450 50  0001 C CNN
+F 1 "+5V" H 6665 2773 50  0000 C CNN
+F 2 "" H 6650 2600 50  0001 C CNN
+F 3 "" H 6650 2600 50  0001 C CNN
+	1    6650 2600
+	1    0    0    -1
+$EndComp
+Wire Wire Line
+	6800 5950 6950 5950
+Wire Wire Line
+	6800 5400 6950 5400
+$Comp
+L Device:R R?
+U 1 1 605D01E3
+P 6950 5250
+F 0 "R?" H 7020 5296 50  0000 L CNN
+F 1 "R" H 7020 5205 50  0000 L CNN
+F 2 "" V 6880 5250 50  0001 C CNN
+F 3 "~" H 6950 5250 50  0001 C CNN
+	1    6950 5250
+	1    0    0    -1
+$EndComp
+Connection ~ 6950 5400
+Wire Wire Line
+	6950 5400 7150 5400
+$Comp
+L Device:R R?
+U 1 1 605D0451
+P 6950 5800
+F 0 "R?" H 7020 5846 50  0000 L CNN
+F 1 "R" H 7020 5755 50  0000 L CNN
+F 2 "" V 6880 5800 50  0001 C CNN
+F 3 "~" H 6950 5800 50  0001 C CNN
+	1    6950 5800
+	1    0    0    -1
+$EndComp
+Connection ~ 6950 5950
+Wire Wire Line
+	6950 5950 7150 5950
+$Comp
+L power:+5V #PWR?
+U 1 1 605D104E
+P 6950 5650
+F 0 "#PWR?" H 6950 5500 50  0001 C CNN
+F 1 "+5V" H 6965 5823 50  0000 C CNN
+F 2 "" H 6950 5650 50  0001 C CNN
+F 3 "" H 6950 5650 50  0001 C CNN
+	1    6950 5650
+	1    0    0    -1
+$EndComp
+$Comp
+L power:+5V #PWR?
+U 1 1 605D1323
+P 6950 5100
+F 0 "#PWR?" H 6950 4950 50  0001 C CNN
+F 1 "+5V" H 6965 5273 50  0000 C CNN
+F 2 "" H 6950 5100 50  0001 C CNN
+F 3 "" H 6950 5100 50  0001 C CNN
+	1    6950 5100
+	1    0    0    -1
+$EndComp
 $EndSCHEMATC

Commit message: ordered it supposedly
Parts:
- C6: renamed from C?; footprint (none) -> Capacitor_SMD:C_0603_1608Metric; LCSC (none) -> C14663
- Q5, Q6: LCSC C31776 -> C2146
- R17, R19: renamed from R?; value R -> 10k; footprint (none) -> Resistor_SMD:R_0603_1608Metric; LCSC (none) -> C25804
- R2, R6: renamed from R?; footprint (none) -> Resistor_SMD:R_0603_1608Metric; LCSC (none) -> C25804
Changed lines of the file:
@@
 F 2 "Package_TO_SOT_SMD:SOT-23" H 4000 1625 50  0001 L CIN
 F 3 "https://assets.nexperia.com/documents/data-sheet/BC846_SER.pdf" H 3800 1700 50  0001 L CNN
-F 4 "C31776" H 3800 1700 50  0001 C CNN "LCSC"
+F 4 "C2146" H 3800 1700 50  0001 C CNN "LCSC"
 	1    3800 1700
 	1    0    0    -1
@@
 F 2 "Package_TO_SOT_SMD:SOT-23" H 4300 4675 50  0001 L CIN
 F 3 "https://assets.nexperia.com/documents/data-sheet/BC846_SER.pdf" H 4100 4750 50  0001 L CNN
-F 4 "C31776" H 4100 4750 50  0001 C CNN "LCSC"
+F 4 "C2146" H 4100 4750 50  0001 C CNN "LCSC"
 	1    4100 4750
 	1    0    0    -1
@@
 	7150 1250 6800 1250
 $Comp
-L Device:C C?
+L Device:C C6
 U 1 1 605BF183
 P 5150 3200
-F 0 "C?" H 5265 3246 50  0000 L CNN
+F 0 "C6" H 5265 3246 50  0000 L CNN
 F 1 ".1uF" H 5265 3155 50  0000 L CNN
-F 2 "" H 5188 3050 50  0001 C CNN
+F 2 "Capacitor_SMD:C_0603_1608Metric" H 5188 3050 50  0001 C CNN
 F 3 "~" H 5150 3200 50  0001 C CNN
+F 4 "C14663" H 5150 3200 50  0001 C CNN "LCSC"
 	1    5150 3200
 	1    0    0    -1
@@
 	6500 2350 6650 2350
 $Comp
-L Device:R R?
+L Device:R R2
 U 1 1 605CB52E
 P 6650 2200
-F 0 "R?" H 6720 2246 50  0000 L CNN
+F 0 "R2" H 6720 2246 50  0000 L CNN
 F 1 "10k" H 6720 2155 50  0000 L CNN
-F 2 "" V 6580 2200 50  0001 C CNN
+F 2 "Resistor_SMD:R_0603_1608Metric" V 6580 2200 50  0001 C CNN
 F 3 "~" H 6650 2200 50  0001 C CNN
+F 4 "C25804" H 6650 2200 50  0001 C CNN "LCSC"
 	1    6650 2200
 	1    0    0    -1
@@
 	6650 2350 6850 2350
 $Comp
-L Device:R R?
+L Device:R R6
 U 1 1 605CB817
 P 6650 2750
-F 0 "R?" H 6720 2796 50  0000 L CNN
+F 0 "R6" H 6720 2796 50  0000 L CNN
 F 1 "10k" H 6720 2705 50  0000 L CNN
-F 2 "" V 6580 2750 50  0001 C CNN
+F 2 "Resistor_SMD:R_0603_1608Metric" V 6580 2750 50  0001 C CNN
 F 3 "~" H 6650 2750 50  0001 C CNN
+F 4 "C25804" H 6650 2750 50  0001 C CNN "LCSC"
 	1    6650 2750
 	1    0    0    -1
@@
 	6650 2900 6850 2900
 $Comp
-L power:+5V #PWR?
+L power:+5V #PWR0132
 U 1 1 605CC9CB
 P 6650 2050
-F 0 "#PWR?" H 6650 1900 50  0001 C CNN
+F 0 "#PWR0132" H 6650 1900 50  0001 C CNN
 F 1 "+5V" H 6665 2223 50  0000 C CNN
 F 2 "" H 6650 2050 50  0001 C CNN
@@
 $EndComp
 $Comp
-L power:+5V #PWR?
+L power:+5V #PWR0137
 U 1 1 605CCCAA
 P 6650 2600
-F 0 "#PWR?" H 6650 2450 50  0001 C CNN
+F 0 "#PWR0137" H 6650 2450 50  0001 C CNN
 F 1 "+5V" H 6665 2773 50  0000 C CNN
 F 2 "" H 6650 2600 50  0001 C CNN
@@
 	6800 5400 6950 5400
 $Comp
-L Device:R R?
+L Device:R R17
 U 1 1 605D01E3
 P 6950 5250
-F 0 "R?" H 7020 5296 50  0000 L CNN
-F 1 "R" H 7020 5205 50  0000 L CNN
-F 2 "" V 6880 5250 50  0001 C CNN
+F 0 "R17" H 7020 5296 50  0000 L CNN
+F 1 "10k" H 7020 5205 50  0000 L CNN
+F 2 "Resistor_SMD:R_0603_1608Metric" V 6880 5250 50  0001 C CNN
 F 3 "~" H 6950 5250 50  0001 C CNN
+F 4 "C25804" H 6950 5250 50  0001 C CNN "LCSC"
 	1    6950 5250
 	1    0    0    -1
@@
 	6950 5400 7150 5400
 $Comp
-L Device:R R?
+L Device:R R19
 U 1 1 605D0451
 P 6950 5800
-F 0 "R?" H 7020 5846 50  0000 L CNN
-F 1 "R" H 7020 5755 50  0000 L CNN
-F 2 "" V 6880 5800 50  0001 C CNN
+F 0 "R19" H 7020 5846 50  0000 L CNN
+F 1 "10k" H 7020 5755 50  0000 L CNN
+F 2 "Resistor_SMD:R_0603_1608Metric" V 6880 5800 50  0001 C CNN
 F 3 "~" H 6950 5800 50  0001 C CNN
+F 4 "C25804" H 6950 5800 50  0001 C CNN "LCSC"
 	1    6950 5800
 	1    0    0    -1
@@
 	6950 5950 7150 5950
 $Comp
-L power:+5V #PWR?
+L power:+5V #PWR0144
 U 1 1 605D104E
 P 6950 5650
-F 0 "#PWR?" H 6950 5500 50  0001 C CNN
+F 0 "#PWR0144" H 6950 5500 50  0001 C CNN
 F 1 "+5V" H 6965 5823 50  0000 C CNN
 F 2 "" H 6950 5650 50  0001 C CNN
@@
 $EndComp
 $Comp
-L power:+5V #PWR?
+L power:+5V #PWR0145
 U 1 1 605D1323
 P 6950 5100
-F 0 "#PWR?" H 6950 4950 50  0001 C CNN
+F 0 "#PWR0145" H 6950 4950 50  0001 C CNN
 F 1 "+5V" H 6965 5273 50  0000 C CNN
 F 2 "" H 6950 5100 50  0001 C CNN

Commit message: containment schematic updated to include experiment & correct voltage on valve mosfets
Parts:
- JFLUID1, JFLUID2: footprint Connector_JST:JST_PH_S3B-PH-K_1x03_P2.00mm_Horizontal -> Connector_JST:JST_PH_B3B-PH-K_1x03_P2.00mm_Vertical
Connections:
- net labels added: sensor_2_hi_expctl, sensor_2_lo_expctl
- net labels removed: sensor_2_hi, sensor_2_lo
Changed lines of the file:
@@
 $Descr A4 11693 8268
 encoding utf-8
-Sheet 2 2
+Sheet 2 3
 Title ""
 Date ""
@@
 F 0 "JFLUID2" H 5430 4342 50  0000 L CNN
 F 1 "Conn_01x03" H 5430 4251 50  0000 L CNN
-F 2 "Connector_JST:JST_PH_S3B-PH-K_1x03_P2.00mm_Horizontal" H 5350 4350 50  0001 C CNN
+F 2 "Connector_JST:JST_PH_B3B-PH-K_1x03_P2.00mm_Vertical" H 5350 4350 50  0001 C CNN
 F 3 "~" H 5350 4350 50  0001 C CNN
 	1    5350 4350
@@
 	1    0    0    -1
 $EndComp
-Text HLabel 7150 5400 2    50   Input ~ 0
-sensor_2_hi
-Text HLabel 7150 5950 2    50   Input ~ 0
-sensor_2_lo
 $Comp
 L Device:R R20
@@
 F 0 "JFLUID1" H 5130 1292 50  0000 L CNN
 F 1 "Conn_01x03" H 5130 1201 50  0000 L CNN
-F 2 "Connector_JST:JST_PH_S3B-PH-K_1x03_P2.00mm_Horizontal" H 5050 1300 50  0001 C CNN
+F 2 "Connector_JST:JST_PH_B3B-PH-K_1x03_P2.00mm_Vertical" H 5050 1300 50  0001 C CNN
 F 3 "~" H 5050 1300 50  0001 C CNN
 	1    5050 1300
@@
 $EndComp
 Connection ~ 6950 5400
-Wire Wire Line
-	6950 5400 7150 5400
 $Comp
 L Device:R R19
@@
 $EndComp
 Connection ~ 6950 5950
-Wire Wire Line
-	6950 5950 7150 5950
 $Comp
 L power:+5V #PWR0144
@@
 	1    0    0    -1
 $EndComp
+Wire Wire Line
+	6950 5400 7150 5400
+Text HLabel 7150 5400 2    50   Input ~ 0
+sensor_2_hi_expctl
+Wire Wire Line
+	6950 5950 7150 5950
+Text HLabel 7150 5950 2    50   Input ~ 0
+sensor_2_lo_expctl
 $EndSCHEMATC
