File: spaceduino/custom.sch (KiCad schematic (older format))
At the start: 0 parts

Commit message: add SD card footprint, PNP-based current mirror
Parts:
- added Q4: BC856BS, Package_TO_SOT_SMD:SOT-363_SC-70-6, symbol Transistor_BJT:BC856BS
- added Q5: BSS84, Package_TO_SOT_SMD:SOT-23, symbol Transistor_FET:BSS84
- added R22: 50m, symbol Device:R
- added R23, R24: 10, symbol Device:R
- added R25: 27, symbol Device:R
- added R26: 10k, symbol Device:R
- added RV1: R_POT, symbol Device:R_POT
- added U8: MPD200A, Spaceduino:MPD200A, symbol Spaceduino_Parts:MPD200A
- added U9: INA226, Package_SO:VSSOP-10_3x3mm_P0.5mm, symbol Analog_ADC:INA226
Connections:
- new net: Q4.1 (E1), R23.2
- new net: Q4.2 (B1), Q4.5 (B2), Q4.6 (C1), R26.2, RV1.2, RV1.3
- new net: Q4.4 (E2), R24.2
- new net: R22.2, R24.1, U9.9 (Vin-)
- new net: R25.1, RV1.1
- new net: Q5.2 (S), R23.1
- new net +5V: Q5.3 (D), R22.1, R26.1, U8.1 (VDD), U9.1 (A1), U9.10 (Vin+), U9.6 (VS)
- new net GND: R25.2, U8.5 (GND), U8.8 (GND), U9.2 (A0), U9.3 (~Alert~), U9.7 (GND)
- new net HV+: U8.10 (HV+)
- new net HV-: U8.6 (HV-)
- new net a3_pump_en: U8.3 (~ENABLE)
- new net experiment: Q4.3 (C2), U9.8 (Vbus)
- new net i2c_scl: U9.5 (SCL)
- new net i2c_sda: U9.4 (SDA)
- no-connect marks 0 -> 2
Other:
- note added: "connect jumpers on mpd200a for\nmaximum power as per datasheet"
