File: spaceduino/spaceduino.sch (KiCad schematic (older format))
At the start: 76 parts, among them J1 USB_B, J2 Micro_SD_Card, J3 JICSP, J4 Conn_02x05_Odd_Even, Q1 BSS84, Q2 BSS84, Q3 BSS84, SW1 SW_SPST, U1 TLV70030_SOT23-5, U2 FT230XS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

Commit message: can i get a go dawgs
Parts:
- C1, C10, C12, C16, C19, C2, C20, C3, C5, C9: LCSC C77055 -> C14663
- C11, C13: LCSC C599690 -> C1653
- C14, C17, C18, C8: LCSC C14860 -> C13585
- C15: LCSC C519421 -> C1595
- C4: LCSC C141215 -> C1848
- D1, D2: LCSC C222352 -> C8598
- D3PWR1, DALERT1, DIND1, DPWR1: LCSC C192676 -> C125086
- DBPWR1, DBPWR2: LCSC C264549 -> C125086
- FB1: LCSC C88995 -> C131463
- R1, R2: LCSC C52199 -> C4410
- R11, R6: LCSC C601102 -> C201301
- R13: LCSC C4502 -> C17936
Changed lines of the file:
@@
 F 3 "~" H 6050 2350 50  0001 C CNN
 F 4 "10uF" H 6050 2350 50  0001 C CNN "Comment"
-F 5 "C14860" H 6050 2350 50  0001 C CNN "LCSC"
+F 5 "C13585" H 6050 2350 50  0001 C CNN "LCSC"
 	1    6050 2350
 	1    0    0    -1
@@
 F 3 "~" H 4900 2500 50  0001 C CNN
 F 4 ".1uF" H 4900 2500 50  0001 C CNN "Comment"
-F 5 "C77055" H 4900 2500 50  0001 C CNN "LCSC"
+F 5 "C14663" H 4900 2500 50  0001 C CNN "LCSC"
 	1    4900 2500
 	1    0    0    -1
@@
 F 3 "~" H 1800 900 50  0001 C CNN
 F 4 ".1uF" H 1800 900 50  0001 C CNN "Comment"
-F 5 "C77055" H 1800 900 50  0001 C CNN "LCSC"
+F 5 "C14663" H 1800 900 50  0001 C CNN "LCSC"
 	1    1800 900
 	1    0    0    -1
@@
 F 3 "~" H 7000 5050 50  0001 C CNN
 F 4 "10uF" H 7000 5050 50  0001 C CNN "Comment"
-F 5 "C14860" H 7000 5050 50  0001 C CNN "LCSC"
+F 5 "C13585" H 7000 5050 50  0001 C CNN "LCSC"
 	1    7000 5050
 	1    0    0    -1
@@
 F 3 "~" H 6000 1250 50  0001 C CNN
 F 4 "1uF" H 6000 1250 50  0001 C CNN "Comment"
-F 5 "C141215" H 6000 1250 50  0001 C CNN "LCSC"
+F 5 "C1848" H 6000 1250 50  0001 C CNN "LCSC"
 	1    6000 1250
 	1    0    0    -1
@@
 F 3 "~" H 4950 1250 50  0001 C CNN
 F 4 ".1uF" H 4950 1250 50  0001 C CNN "Comment"
-F 5 "C77055" H 4950 1250 50  0001 C CNN "LCSC"
+F 5 "C14663" H 4950 1250 50  0001 C CNN "LCSC"
 	1    4950 1250
 	1    0    0    -1
@@
 F 3 "~" H 2500 650 50  0001 C CNN
 F 4 ".1uF" H 2500 650 50  0001 C CNN "Comment"
-F 5 "C77055" H 2500 650 50  0001 C CNN "LCSC"
+F 5 "C14663" H 2500 650 50  0001 C CNN "LCSC"
 	1    2500 650
 	1    0    0    -1
@@
 F 3 "~" H 4850 3950 50  0001 C CNN
 F 4 ".1uF" H 4850 3950 50  0001 C CNN "Comment"
-F 5 "C77055" H 4850 3950 50  0001 C CNN "LCSC"
+F 5 "C14663" H 4850 3950 50  0001 C CNN "LCSC"
 	1    4850 3950
 	1    0    0    -1
@@
 F 3 "~" H 4350 1550 50  0001 C CNN
 F 4 ".1uF" H 4350 1550 50  0001 C CNN "Comment"
-F 5 "C77055" H 4350 1550 50  0001 C CNN "LCSC"
+F 5 "C14663" H 4350 1550 50  0001 C CNN "LCSC"
 	1    4350 1550
 	0    1    1    0
@@
 F 2 "LED_SMD:LED_1206_3216Metric" H 600 5550 50  0001 C CNN
 F 3 "~" H 600 5550 50  0001 C CNN
-F 4 "C192676" H 600 5550 50  0001 C CNN "LCSC"
+F 4 "C125086" H 600 5550 50  0001 C CNN "LCSC"
 	1    600  5550
 	0    -1   -1   0
@@
 F 3 "~" H 1000 5250 50  0001 C CNN
 F 4 "470R" H 1000 5250 50  0001 C CNN "Comment"
-F 5 "C4502" H 1000 5250 50  0001 C CNN "LCSC"
+F 5 "C17936" H 1000 5250 50  0001 C CNN "LCSC"
 	1    1000 5250
 	1    0    0    -1
@@
 F 2 "LED_SMD:LED_1206_3216Metric" H 1000 5550 50  0001 C CNN
 F 3 "~" H 1000 5550 50  0001 C CNN
-F 4 "C192676" H 1000 5550 50  0001 C CNN "LCSC"
+F 4 "C125086" H 1000 5550 50  0001 C CNN "LCSC"
 	1    1000 5550
 	0    -1   -1   0
@@
 F 2 "LED_SMD:LED_1206_3216Metric" H 2100 5550 50  0001 C CNN
 F 3 "~" H 2100 5550 50  0001 C CNN
-F 4 "C192676" H 2100 5550 50  0001 C CNN "LCSC"
+F 4 "C125086" H 2100 5550 50  0001 C CNN "LCSC"
 	1    2100 5550
 	0    -1   -1   0
@@
 F 3 "~" H 4250 1050 50  0001 C CNN
 F 4 "1K" H 4250 1050 50  0001 C CNN "Comment"
-F 5 "C52199" H 4250 1050 50  0001 C CNN "LCSC"
+F 5 "C4410" H 4250 1050 50  0001 C CNN "LCSC"
 	1    4250 1050
 	0    1    1    0
@@
 F 3 "~" H 4250 1150 50  0001 C CNN
 F 4 "1K" H 4250 1150 50  0001 C CNN "Comment"
-F 5 "C52199" H 4250 1150 50  0001 C CNN "LCSC"
+F 5 "C4410" H 4250 1150 50  0001 C CNN "LCSC"
 	1    4250 1150
 	0    1    1    0
@@
 F 2 "Diode_SMD:D_SOD-123" H 2000 3300 50  0001 C CNN
 F 3 "~" H 2000 3300 50  0001 C CNN
-F 4 "C222352" H 2000 3300 50  0001 C CNN "LCSC"
+F 4 "C8598" H 2000 3300 50  0001 C CNN "LCSC"
 	1    2000 3300
 	-1   0    0    1
@@
 F 3 "~" H 2100 3900 50  0001 C CNN
 F 4 "1.5nF" H 2100 3900 50  0001 C CNN "Comment"
-F 5 "C519421" H 2100 3900 50  0001 C CNN "LCSC"
+F 5 "C1595" H 2100 3900 50  0001 C CNN "LCSC"
 	1    2100 3900
 	1    0    0    -1
@@
 F 3 "~" H 2750 3850 50  0001 C CNN
 F 4 "10uF" H 2750 3850 50  0001 C CNN "Comment"
-F 5 "C14860" H 2750 3850 50  0001 C CNN "LCSC"
+F 5 "C13585" H 2750 3850 50  0001 C CNN "LCSC"
 	1    2750 3850
 	1    0    0    -1
@@
 F 3 "~" H 600 3600 50  0001 C CNN
 F 4 ".1uF" H 600 3600 50  0001 C CNN "Comment"
-F 5 "C77055" H 600 3600 50  0001 C CNN "LCSC"
+F 5 "C14663" H 600 3600 50  0001 C CNN "LCSC"
 	1    600  3600
 	1    0    0    -1
@@
 F 2 "LED_SMD:LED_1206_3216Metric" H 2500 5550 50  0001 C CNN
 F 3 "~" H 2500 5550 50  0001 C CNN
-F 4 "C192676" H 2500 5550 50  0001 C CNN "LCSC"
+F 4 "C125086" H 2500 5550 50  0001 C CNN "LCSC"
 	1    2500 5550
 	0    -1   -1   0
@@
 F 3 "~" H 7850 4850 50  0001 C CNN
 F 4 "50mR" H 7850 4850 50  0001 C CNN "Comment"
-F 5 "C601102" H 7850 4850 50  0001 C CNN "LCSC"
+F 5 "C201301" H 7850 4850 50  0001 C CNN "LCSC"
 	1    7850 4850
 	0    1    1    0
@@
 F 3 "~" H 4600 3600 50  0001 C CNN
 F 4 "22pF" H 4600 3600 50  0001 C CNN "Comment"
-F 5 "C599690" H 4600 3600 50  0001 C CNN "LCSC"
+F 5 "C1653" H 4600 3600 50  0001 C CNN "LCSC"
 	1    4600 3600
 	0    1    1    0
@@
 F 3 "~" H 4600 3300 50  0001 C CNN
 F 4 "22pF" H 4600 3300 50  0001 C CNN "Comment"
-F 5 "C599690" H 4600 3300 50  0001 C CNN "LCSC"
+F 5 "C1653" H 4600 3300 50  0001 C CNN "LCSC"
 	1    4600 3300
 	0    1    1    0
@@
 F 2 "Diode_SMD:D_SOD-123" H 4700 3000 50  0001 C CNN
 F 3 "~" H 4700 3000 50  0001 C CNN
-F 4 "C222352" H 4700 3000 50  0001 C CNN "LCSC"
+F 4 "C8598" H 4700 3000 50  0001 C CNN "LCSC"
 	1    4700 3000
 	0    1    1    0
@@
 F 3 "~" H 3200 3300 50  0001 C CNN
 F 4 "50mR" H 3200 3300 50  0001 C CNN "Comment"
-F 5 "C601102" H 3200 3300 50  0001 C CNN "LCSC"
+F 5 "C201301" H 3200 3300 50  0001 C CNN "LCSC"
 	1    3200 3300
 	0    1    1    0
@@
 F 2 "Inductor_SMD:L_1206_3216Metric" V 6930 4250 50  0001 C CNN
 F 3 "~" H 7000 4250 50  0001 C CNN
-F 4 "C88995" H 7000 4250 50  0001 C CNN "LCSC"
+F 4 "C131463" H 7000 4250 50  0001 C CNN "LCSC"
 	1    7000 4250
 	1    0    0    -1
@@
 F 3 "~" H 750 7100 50  0001 C CNN
 F 4 ".1uF" H 750 7100 50  0001 C CNN "Comment"
-F 5 "C77055" H 750 7100 50  0001 C CNN "LCSC"
+F 5 "C14663" H 750 7100 50  0001 C CNN "LCSC"
 	1    750  7100
 	1    0    0    -1
@@
 F 3 "~" H 10150 6050 50  0001 C CNN
 F 4 "10uF" H 10150 6050 50  0001 C CNN "Comment"
-F 5 "C14860" H 10150 6050 50  0001 C CNN "LCSC"
+F 5 "C13585" H 10150 6050 50  0001 C CNN "LCSC"
 	1    10150 6050
 	1    0    0    -1
@@
 F 3 "~" H 1150 7100 50  0001 C CNN
 F 4 ".1uF" H 1150 7100 50  0001 C CNN "Comment"
-F 5 "C77055" H 1150 7100 50  0001 C CNN "LCSC"
+F 5 "C14663" H 1150 7100 50  0001 C CNN "LCSC"
 	1    1150 7100
 	1    0    0    -1
@@
 F 3 "~" H 6650 850 50  0001 C CNN
 F 4 ".1uF" H 6650 850 50  0001 C CNN "Comment"
-F 5 "C77055" H 6650 850 50  0001 C CNN "LCSC"
+F 5 "C14663" H 6650 850 50  0001 C CNN "LCSC"
 	1    6650 850
 	1    0    0    -1
@@
 F 2 "LED_SMD:LED_1206_3216Metric" H 1700 5550 50  0001 C CNN
 F 3 "~" H 1700 5550 50  0001 C CNN
-F 4 "C264549" H 1700 5550 50  0001 C CNN "LCSC"
+F 4 "C125086" H 1700 5550 50  0001 C CNN "LCSC"
 	1    1700 5550
 	0    -1   -1   0
@@
 F 2 "LED_SMD:LED_1206_3216Metric" H 1700 5850 50  0001 C CNN
 F 3 "~" H 1700 5850 50  0001 C CNN
-F 4 "C264549" H 1700 5850 50  0001 C CNN "LCSC"
+F 4 "C125086" H 1700 5850 50  0001 C CNN "LCSC"
 	1    1700 5850
 	0    -1   -1   0

Commit message: ordered it supposedly
Parts:
- C12: value .1uF -> 10uF; footprint Capacitor_SMD:C_0603_1608Metric -> Capacitor_SMD:C_1206_3216Metric; LCSC C14663 -> C13585
- D3PWR1, DBPWR1, DBPWR2, DIND1, DPWR1: footprint LED_SMD:LED_1206_3216Metric -> LED_SMD:LED_0603_1608Metric; LCSC C125086 -> C72041
- DALERT1: footprint LED_SMD:LED_1206_3216Metric -> LED_SMD:LED_0603_1608Metric; LCSC C125086 -> C2286
- Q1, Q2, Q3: LCSC C508197 -> C10487
- R10: footprint Resistor_SMD:R_1206_3216Metric -> Resistor_SMD:R_0603_1608Metric; LCSC C18007 -> C23147
- R12, R15, R16, R9: footprint Resistor_SMD:R_1206_3216Metric -> Resistor_SMD:R_0603_1608Metric; LCSC C26030 -> C22843
- R14: footprint Resistor_SMD:R_1206_3216Metric -> Resistor_SMD:R_0603_1608Metric; LCSC C18028 -> C23189
- R17, R18: footprint Resistor_SMD:R_1206_3216Metric -> Resistor_SMD:R_0603_1608Metric; LCSC C26032 -> C22978
- R3, R4: footprint Resistor_SMD:R_1206_3216Metric -> Resistor_SMD:R_0603_1608Metric; LCSC C17946 -> C25190
- R7: footprint Resistor_SMD:R_1206_3216Metric -> Resistor_SMD:R_0603_1608Metric; LCSC C34847 -> C22797
Changed lines of the file:
@@
 F 0 "R3" V 1793 1350 50  0000 C CNN
 F 1 "27" V 1884 1350 50  0000 C CNN
-F 2 "Resistor_SMD:R_1206_3216Metric" V 1930 1350 50  0001 C CNN
+F 2 "Resistor_SMD:R_0603_1608Metric" V 1930 1350 50  0001 C CNN
 F 3 "~" H 2000 1350 50  0001 C CNN
 F 4 "27R" H 2000 1350 50  0001 C CNN "Comment"
-F 5 "C17946" H 2000 1350 50  0001 C CNN "LCSC"
+F 5 "C25190" H 2000 1350 50  0001 C CNN "LCSC"
 	1    2000 1350
 	0    1    1    0
@@
 F 0 "R4" V 2100 1450 50  0000 C CNN
 F 1 "27" V 2200 1450 50  0000 C CNN
-F 2 "Resistor_SMD:R_1206_3216Metric" V 1930 1450 50  0001 C CNN
+F 2 "Resistor_SMD:R_0603_1608Metric" V 1930 1450 50  0001 C CNN
 F 3 "~" H 2000 1450 50  0001 C CNN
 F 4 "27R" H 2000 1450 50  0001 C CNN "Comment"
-F 5 "C17946" H 2000 1450 50  0001 C CNN "LCSC"
+F 5 "C25190" H 2000 1450 50  0001 C CNN "LCSC"
 	1    2000 1450
 	0    1    1    0
@@
 F 0 "R12" H 670 5296 50  0000 L CNN
 F 1 "1.5k" H 670 5205 50  0000 L CNN
-F 2 "Resistor_SMD:R_1206_3216Metric" V 530 5250 50  0001 C CNN
+F 2 "Resistor_SMD:R_0603_1608Metric" V 530 5250 50  0001 C CNN
 F 3 "~" H 600 5250 50  0001 C CNN
 F 4 "1.5K" H 600 5250 50  0001 C CNN "Comment"
-F 5 "C26030" H 600 5250 50  0001 C CNN "LCSC"
+F 5 "C22843" H 600 5250 50  0001 C CNN "LCSC"
 	1    600  5250
 	1    0    0    -1
@@
 F 0 "DPWR1" V 639 5433 50  0000 R CNN
 F 1 "LED" V 548 5433 50  0000 R CNN
-F 2 "LED_SMD:LED_1206_3216Metric" H 600 5550 50  0001 C CNN
+F 2 "LED_SMD:LED_0603_1608Metric" H 600 5550 50  0001 C CNN
 F 3 "~" H 600 5550 50  0001 C CNN
-F 4 "C125086" H 600 5550 50  0001 C CNN "LCSC"
+F 4 "C72041" H 600 5550 50  0001 C CNN "LCSC"
 	1    600  5550
 	0    -1   -1   0
@@
 F 0 "D3PWR1" V 1039 5433 50  0000 R CNN
 F 1 "LED" V 948 5433 50  0000 R CNN
-F 2 "LED_SMD:LED_1206_3216Metric" H 1000 5550 50  0001 C CNN
+F 2 "LED_SMD:LED_0603_1608Metric" H 1000 5550 50  0001 C CNN
 F 3 "~" H 1000 5550 50  0001 C CNN
-F 4 "C125086" H 1000 5550 50  0001 C CNN "LCSC"
+F 4 "C72041" H 1000 5550 50  0001 C CNN "LCSC"
 	1    1000 5550
 	0    -1   -1   0
@@
 F 0 "R14" H 1770 5296 50  0000 L CNN
 F 1 "5.6k" H 1770 5205 50  0000 L CNN
-F 2 "Resistor_SMD:R_1206_3216Metric" V 1630 5250 50  0001 C CNN
+F 2 "Resistor_SMD:R_0603_1608Metric" V 1630 5250 50  0001 C CNN
 F 3 "~" H 1700 5250 50  0001 C CNN
 F 4 "5K6" H 1700 5250 50  0001 C CNN "Comment"
-F 5 "C18028" H 1700 5250 50  0001 C CNN "LCSC"
+F 5 "C23189" H 1700 5250 50  0001 C CNN "LCSC"
 	1    1700 5250
 	1    0    0    -1
@@
 F 0 "R15" H 2170 5296 50  0000 L CNN
 F 1 "1.5k" H 2170 5205 50  0000 L CNN
-F 2 "Resistor_SMD:R_1206_3216Metric" V 2030 5250 50  0001 C CNN
+F 2 "Resistor_SMD:R_0603_1608Metric" V 2030 5250 50  0001 C CNN
 F 3 "~" H 2100 5250 50  0001 C CNN
 F 4 "1.5K" H 2100 5250 50  0001 C CNN "Comment"
-F 5 "C26030" H 2100 5250 50  0001 C CNN "LCSC"
+F 5 "C22843" H 2100 5250 50  0001 C CNN "LCSC"
 	1    2100 5250
 	1    0    0    -1
@@
 F 0 "DIND1" V 2139 5433 50  0000 R CNN
 F 1 "LED" V 2048 5433 50  0000 R CNN
-F 2 "LED_SMD:LED_1206_3216Metric" H 2100 5550 50  0001 C CNN
+F 2 "LED_SMD:LED_0603_1608Metric" H 2100 5550 50  0001 C CNN
 F 3 "~" H 2100 5550 50  0001 C CNN
-F 4 "C125086" H 2100 5550 50  0001 C CNN "LCSC"
+F 4 "C72041" H 2100 5550 50  0001 C CNN "LCSC"
 	1    2100 5550
 	0    -1   -1   0
@@
 F 0 "R7" H 2570 3496 50  0000 L CNN
 F 1 "13k" H 2570 3405 50  0000 L CNN
-F 2 "Resistor_SMD:R_1206_3216Metric" V 2430 3450 50  0001 C CNN
+F 2 "Resistor_SMD:R_0603_1608Metric" V 2430 3450 50  0001 C CNN
 F 3 "~" H 2500 3450 50  0001 C CNN
 F 4 "13K" H 2500 3450 50  0001 C CNN "Comment"
-F 5 "C34847" H 2500 3450 50  0001 C CNN "LCSC"
+F 5 "C22797" H 2500 3450 50  0001 C CNN "LCSC"
 	1    2500 3450
 	1    0    0    -1
@@
 F 0 "R9" H 2570 4246 50  0000 L CNN
 F 1 "1.5k" H 2570 4155 50  0000 L CNN
-F 2 "Resistor_SMD:R_1206_3216Metric" V 2430 4200 50  0001 C CNN
+F 2 "Resistor_SMD:R_0603_1608Metric" V 2430 4200 50  0001 C CNN
 F 3 "~" H 2500 4200 50  0001 C CNN
 F 4 "1.5K" H 2500 4200 50  0001 C CNN "Comment"
-F 5 "C26030" H 2500 4200 50  0001 C CNN "LCSC"
+F 5 "C22843" H 2500 4200 50  0001 C CNN "LCSC"
 	1    2500 4200
 	1    0    0    -1
@@
 P 600 3600
 F 0 "C12" H 715 3646 50  0000 L CNN
-F 1 ".1uF" H 715 3555 50  0000 L CNN
-F 2 "Capacitor_SMD:C_0603_1608Metric" H 638 3450 50  0001 C CNN
+F 1 "10uF" H 715 3555 50  0000 L CNN
+F 2 "Capacitor_SMD:C_1206_3216Metric" H 638 3450 50  0001 C CNN
 F 3 "~" H 600 3600 50  0001 C CNN
 F 4 ".1uF" H 600 3600 50  0001 C CNN "Comment"
-F 5 "C14663" H 600 3600 50  0001 C CNN "LCSC"
+F 5 "C13585" H 600 3600 50  0001 C CNN "LCSC"
 	1    600  3600
 	1    0    0    -1
@@
 F 0 "R16" H 2570 5296 50  0000 L CNN
 F 1 "1.5k" H 2570 5205 50  0000 L CNN
-F 2 "Resistor_SMD:R_1206_3216Metric" V 2430 5250 50  0001 C CNN
+F 2 "Resistor_SMD:R_0603_1608Metric" V 2430 5250 50  0001 C CNN
 F 3 "~" H 2500 5250 50  0001 C CNN
 F 4 "1.5K" H 2500 5250 50  0001 C CNN "Comment"
-F 5 "C26030" H 2500 5250 50  0001 C CNN "LCSC"
+F 5 "C22843" H 2500 5250 50  0001 C CNN "LCSC"
 	1    2500 5250
 	1    0    0    -1
@@
 F 0 "DALERT1" V 2539 5433 50  0000 R CNN
 F 1 "LED" V 2448 5433 50  0000 R CNN
-F 2 "LED_SMD:LED_1206_3216Metric" H 2500 5550 50  0001 C CNN
+F 2 "LED_SMD:LED_0603_1608Metric" H 2500 5550 50  0001 C CNN
 F 3 "~" H 2500 5550 50  0001 C CNN
-F 4 "C125086" H 2500 5550 50  0001 C CNN "LCSC"
+F 4 "C2286" H 2500 5550 50  0001 C CNN "LCSC"
 	1    2500 5550
 	0    -1   -1   0
@@
 F 2 "Package_TO_SOT_SMD:SOT-23" H 9000 3575 50  0001 L CIN
 F 3 "http://assets.nexperia.com/documents/data-sheet/BSS84.pdf" H 8800 3650 50  0001 L CNN
-F 4 "C508197" H 8800 3650 50  0001 C CNN "LCSC"
+F 4 "C10487" H 8800 3650 50  0001 C CNN "LCSC"
 	1    8800 3650
 	0    1    -1   0
@@
 F 2 "Package_TO_SOT_SMD:SOT-23" H 8500 3975 50  0001 L CIN
 F 3 "http://assets.nexperia.com/documents/data-sheet/BSS84.pdf" H 8300 4050 50  0001 L CNN
-F 4 "C508197" H 8300 4050 50  0001 C CNN "LCSC"
+F 4 "C10487" H 8300 4050 50  0001 C CNN "LCSC"
 	1    8300 4050
 	0    1    -1   0
@@
 F 0 "R10" H 10620 6096 50  0000 L CNN
 F 1 "36k" H 10620 6005 50  0000 L CNN
-F 2 "Resistor_SMD:R_1206_3216Metric" V 10480 6050 50  0001 C CNN
+F 2 "Resistor_SMD:R_0603_1608Metric" V 10480 6050 50  0001 C CNN
 F 3 "~" H 10550 6050 50  0001 C CNN
 F 4 "36K" H 10550 6050 50  0001 C CNN "Comment"
-F 5 "C18007" H 10550 6050 50  0001 C CNN "LCSC"
+F 5 "C23147" H 10550 6050 50  0001 C CNN "LCSC"
 	1    10550 6050
 	1    0    0    -1
@@
 F 0 "R17" H 7320 2996 50  0000 L CNN
 F 1 "3.3k" H 7320 2905 50  0000 L CNN
-F 2 "Resistor_SMD:R_1206_3216Metric" V 7180 2950 50  0001 C CNN
+F 2 "Resistor_SMD:R_0603_1608Metric" V 7180 2950 50  0001 C CNN
 F 3 "~" H 7250 2950 50  0001 C CNN
 F 4 "3K3" H 7250 2950 50  0001 C CNN "Comment"
-F 5 "C26032" H 7250 2950 50  0001 C CNN "LCSC"
+F 5 "C22978" H 7250 2950 50  0001 C CNN "LCSC"
 	1    7250 2950
 	1    0    0    -1
@@
 F 0 "R18" H 7820 3096 50  0000 L CNN
 F 1 "3.3k" H 7820 3005 50  0000 L CNN
-F 2 "Resistor_SMD:R_1206_3216Metric" V 7680 3050 50  0001 C CNN
+F 2 "Resistor_SMD:R_0603_1608Metric" V 7680 3050 50  0001 C CNN
 F 3 "~" H 7750 3050 50  0001 C CNN
 F 4 "3K3" H 7750 3050 50  0001 C CNN "Comment"
-F 5 "C26032" H 7750 3050 50  0001 C CNN "LCSC"
+F 5 "C22978" H 7750 3050 50  0001 C CNN "LCSC"
 	1    7750 3050
 	1    0    0    -1
@@
 F 2 "Package_TO_SOT_SMD:SOT-23" H 10250 5075 50  0001 L CIN
 F 3 "http://assets.nexperia.com/documents/data-sheet/BSS84.pdf" H 10050 5150 50  0001 L CNN
-F 4 "C508197" H 10050 5150 50  0001 C CNN "LCSC"
+F 4 "C10487" H 10050 5150 50  0001 C CNN "LCSC"
 	1    10050 5150
 	1    0    0    1
@@
 F 0 "DBPWR1" V 1739 5433 50  0000 R CNN
 F 1 "LED" V 1648 5433 50  0000 R CNN
-F 2 "LED_SMD:LED_1206_3216Metric" H 1700 5550 50  0001 C CNN
+F 2 "LED_SMD:LED_0603_1608Metric" H 1700 5550 50  0001 C CNN
 F 3 "~" H 1700 5550 50  0001 C CNN
-F 4 "C125086" H 1700 5550 50  0001 C CNN "LCSC"
+F 4 "C72041" H 1700 5550 50  0001 C CNN "LCSC"
 	1    1700 5550
 	0    -1   -1   0
@@
 F 0 "DBPWR2" V 1739 5732 50  0000 R CNN
 F 1 "LED" V 1648 5732 50  0000 R CNN
-F 2 "LED_SMD:LED_1206_3216Metric" H 1700 5850 50  0001 C CNN
+F 2 "LED_SMD:LED_0603_1608Metric" H 1700 5850 50  0001 C CNN
 F 3 "~" H 1700 5850 50  0001 C CNN
-F 4 "C125086" H 1700 5850 50  0001 C CNN "LCSC"
+F 4 "C72041" H 1700 5850 50  0001 C CNN "LCSC"
 	1    1700 5850
 	0    -1   -1   0
